File: BusIndicator.kicad_pcb (KiCad board)
At the start: 2 copper layers, 40 x 46.4 mm, 28 parts, among them J1 Input, SW1 SW_DIP_x08, U1 74AHC244

Commit message: First completely routed version of the Board, ready for review.
Parts:
- D1: value B0 -> LED; footprint Resistor_SMD:R_0805_2012Metric_Pad1.20x1.40mm_HandSolder -> LED_SMD:LED_0805_2012Metric_Pad1.15x1.40mm_HandSolder
- D2: value B1 -> LED; footprint Resistor_SMD:R_0805_2012Metric_Pad1.20x1.40mm_HandSolder -> LED_SMD:LED_0805_2012Metric_Pad1.15x1.40mm_HandSolder
- D3: value B2 -> LED; footprint Resistor_SMD:R_0805_2012Metric_Pad1.20x1.40mm_HandSolder -> LED_SMD:LED_0805_2012Metric_Pad1.15x1.40mm_HandSolder
- D4: value B3 -> LED; footprint Resistor_SMD:R_0805_2012Metric_Pad1.20x1.40mm_HandSolder -> LED_SMD:LED_0805_2012Metric_Pad1.15x1.40mm_HandSolder
- D5: value B4 -> LED; footprint Resistor_SMD:R_0805_2012Metric_Pad1.20x1.40mm_HandSolder -> LED_SMD:LED_0805_2012Metric_Pad1.15x1.40mm_HandSolder
- D6: value B5 -> LED; footprint Resistor_SMD:R_0805_2012Metric_Pad1.20x1.40mm_HandSolder -> LED_SMD:LED_0805_2012Metric_Pad1.15x1.40mm_HandSolder
- D7: value B6 -> LED; footprint Resistor_SMD:R_0805_2012Metric_Pad1.20x1.40mm_HandSolder -> LED_SMD:LED_0805_2012Metric_Pad1.15x1.40mm_HandSolder
- D8: value B7 -> LED; footprint Resistor_SMD:R_0805_2012Metric_Pad1.20x1.40mm_HandSolder -> LED_SMD:LED_0805_2012Metric_Pad1.15x1.40mm_HandSolder
- moved SW1 1.03 mm to (65.2, 76.4)
- moved R10 1.03 mm to (45.9, 73.0)
- moved R11 1.03 mm to (45.9, 76.5)
- moved R12 1.03 mm to (45.9, 79.5)
- moved R13 1.03 mm to (50.4, 69.5)
- moved R14 1.03 mm to (50.4, 73.0)
- moved R15 1.03 mm to (50.4, 76.5)
- moved R16 1.03 mm to (50.4, 79.5)
- moved R9 1.03 mm to (45.9, 69.5)
- turned R1 to 180 degrees
- turned R2 to 180 degrees
- turned R3 to 180 degrees
- turned R4 to 180 degrees
- turned R5 to 180 degrees
- turned R6 to 180 degrees
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Routing:
- net GND: track 185.8 -> 20.0 mm, vias 0 -> 19
- net Net-(J1-Pin_5): track 140.1 -> 54.2 mm, vias 0 -> 4
- net Net-(J1-Pin_7): track 149.5 -> 66.1 mm, vias 0 -> 1
- net Net-(J1-Pin_4): track 103.2 -> 60.1 mm, vias 0 -> 3
- net Net-(J1-Pin_6): track 79.0 -> 40.6 mm, vias 2 -> 1
- net Net-(J1-Pin_3): track 110.9 -> 74.0 mm, vias 0 -> 3
- net Net-(J1-Pin_10): track 64.8 -> 29.0 mm, vias 0 -> 1
- net Net-(J1-Pin_8): track 88.3 -> 56.2 mm, vias 0 -> 1
- net 5V: track 115.2 -> 94.8 mm
- net Net-(D5-A): track 35.9 -> 18.5 mm
- net Net-(D3-A): track 26.7 -> 10.8 mm, vias 0 -> 1
- net Net-(D7-K): track 19.3 -> 4.30 mm
- net Net-(D7-A): track 31.8 -> 16.9 mm, vias 1 -> 0
- net Net-(J1-Pin_9): track 59.2 -> 44.4 mm, vias 2 -> 1
- net Net-(D8-A): track 27.1 -> 16.0 mm, vias 1 -> 0
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- added copper zone on B.Cu, net GND

Commit message: Changed DIP switch to THT footprint.
Parts:
- SW1: footprint Button_Switch_SMD:SW_DIP_SPSTx08_Slide_6.7x21.88mm_W6.73mm_P2.54mm_LowProfile_JPin -> Package_DIP:DIP-16_W7.62mm_Socket_LongPads
- moved SW1 10.1 mm to (74.2, 71.9)
Routing:
- net 5V: track 94.8 -> 83.2 mm
- net GND: track 20.0 -> 13.6 mm, vias 19 -> 17
- net Net-(J1-Pin_3): track 74.0 -> 77.2 mm, vias 3 -> 1
- net Net-(J1-Pin_9): track 44.4 -> 42.7 mm, vias 1 -> 0
- net Net-(D7-A): track 16.9 -> 18.5 mm
- net Net-(J1-Pin_10): track 29.0 -> 27.5 mm, vias 1 -> 0
- net Net-(D8-A): track 16.0 -> 17.3 mm
- net Net-(J1-Pin_4): track 60.1 -> 61.3 mm, vias 3 -> 2
- net Net-(J1-Pin_8): track 56.2 -> 55.2 mm
- net Net-(J1-Pin_5): track 54.2 -> 55.1 mm, vias 4 -> 2
- net Net-(J1-Pin_6): track 40.6 -> 40.3 mm, vias 1 -> 0
- net Net-(D6-A): track 17.6 -> 17.9 mm, vias 0 -> 2
- net Net-(D4-A): vias 1 -> 0
- net Net-(D3-A): vias 1 -> 0
